Commit message: Update files

File: rhacobot_description/urdf/include/materials.xacro (robot description, xacro)
@@ -13,4 +13,10 @@
     <color rgba="1 0.6 0 1" />
   </material>
+  <material name="blue">
+    <color rgba="0 0 1 1" />
+  </material>
+  <material name="green">
+    <color rgba="0 1 0 1" />
+  </material>
   <material name="white">
     <color rgba="1 1 1 1" />

File: rhacobot_description/urdf/rhacobot.urdf.xacro (robot description, xacro)
@@ -6,31 +6,31 @@
   <xacro:arg name="ifname" default="can0" />
  <!-- Import Rviz colors -->
-    <xacro:include filename="$(find gyrosse_description)/urdf/include/materials.xacro" />
+    <xacro:include filename="$(find rhacobot_description)/urdf/include/materials.xacro" />
     <!-- Import Rhacobot Macro -->
-    <xacro:include filename="$(find gyrosse_description)/urdf/rhacobot.joints_links.xacro" />
-    <!-- Import Rhacobot ros2_control description -->
-    <xacro:include filename="$(find gyrosse_description)/urdf/rhacobot.ros2_control.xacro"/>
+    <xacro:include filename="$(find rhacobot_description)/urdf/rhacobot.joints_links.xacro" />
     <link name="base_link"/>
     <!-- Geometry Rhacobot description -->
     <xacro:chassis name="$(arg prefix)chassis"/>
     <xacro:wheel name="$(arg prefix)right_wheel"
-                joint_origin_xyz="0 -0.1905  0"
+                joint_origin_xyz="0 -0.1645  0"
                 joint_rpy="0 0 ${pi}"/>
     <xacro:wheel name="$(arg prefix)left_wheel"
-                joint_origin_xyz="0 0.1905 0"
+                joint_origin_xyz="0 0.1645 0"
                 joint_rpy="0 0 0"/>
-    <xacro:motor_flywheel name="$(arg prefix)motor_flywheel_right"
-                    joint_origin_xyz="0 -0.0825 0"
-                    joint_rpy="0 0 0"/>
-    <xacro:motor_flywheel name="$(arg prefix)motor_flywheel_left"
-                    joint_origin_xyz="0 0.0825 0 "
-                    joint_rpy="0 0 ${pi}"/>
-    <xacro:flywheel name="$(arg prefix)flywheel_right"
-                joint_origin_xyz="0 -0.0825  0"
+    <xacro:tail_joint_a name="$(arg prefix)tail_joint_a"
+                joint_origin_xyz="-0.185 0 -0.0335"
+                joint_rpy="0 0 ${pi}"/>
+    <xacro:tail_joint_b name="$(arg prefix)tail_joint_b"
+                joint_origin_xyz="0 0 0.079"
                 joint_rpy="0 0 0"/>
-    <xacro:flywheel name="$(arg prefix)flywheel_left"
-                joint_origin_xyz="0 0.0825  0"
-                joint_rpy="0 0 ${pi}"/>
-    <xacro:ros2_control name="$(arg name)"
+    <xacro:tail_joint_c name="$(arg prefix)tail_joint_c"
+                joint_origin_xyz="0.25 0 0"
+                joint_rpy="0 0 0"/>
+    <xacro:tail_wheel name="$(arg prefix)tail_wheel"
+                joint_origin_xyz="0.257252 0 0.029622"
+                joint_rpy="0 0 0"/>
+    <!-- Import Rhacobot ros2_control description -->
+    <xacro:include filename="$(find rhacobot_description)/urdf/rhacobot.ros2_control.xacro"/>
+        <xacro:ros2_control name="$(arg name)"
                 prefix="$(arg prefix)"
                 ifname="$(arg ifname)"/>
