Commit message: CleanUp code

File: rhacobot_description/urdf/rhacobot.urdf.xacro (robot description, xacro)
@@ -2,36 +2,18 @@
 <robot xmlns:xacro="http://www.ros.org/wiki/xacro" name="rhacobot_urdf">
     <!-- parameters -->
-  <xacro:arg name="name" default="rhacobot" />
-  <xacro:arg name="prefix" default="" />
-  <xacro:arg name="ifname" default="can0" />
- <!-- Import Rviz colors -->
-    <xacro:include filename="$(find rhacobot_description)/urdf/include/materials.xacro" />
-    <!-- Import Rhacobot Macro -->
-    <xacro:include filename="$(find rhacobot_description)/urdf/rhacobot.joints_links.xacro" />
-    <link name="base_link"/>
-    <!-- Geometry Rhacobot description -->
-    <xacro:chassis name="$(arg prefix)chassis"/>
-    <xacro:wheel name="$(arg prefix)right_wheel"
-                joint_origin_xyz="0 -0.1645  0"
-                joint_rpy="0 0 ${pi}"/>
-    <xacro:wheel name="$(arg prefix)left_wheel"
-                joint_origin_xyz="0 0.1645 0"
-                joint_rpy="0 0 0"/>
-    <xacro:tail_joint_a name="$(arg prefix)tail_joint_a"
-                joint_origin_xyz="-0.185 0 -0.0335"
-                joint_rpy="0 0 ${pi}"/>
-    <xacro:tail_joint_b name="$(arg prefix)tail_joint_b"
-                joint_origin_xyz="0 0 0.079"
-                joint_rpy="0 0 0"/>
-    <xacro:tail_joint_c name="$(arg prefix)tail_joint_c"
-                joint_origin_xyz="0.25 0 0"
-                joint_rpy="0 0 0"/>
-    <xacro:tail_wheel name="$(arg prefix)tail_wheel"
-                joint_origin_xyz="0.257252 0 0.029622"
-                joint_rpy="0 0 0"/>
-    <!-- Import Rhacobot ros2_control description -->
-    <xacro:include filename="$(find rhacobot_description)/urdf/rhacobot.ros2_control.xacro"/>
-        <xacro:ros2_control name="$(arg name)"
-                prefix="$(arg prefix)"
-                ifname="$(arg ifname)"/>
+  <xacro:arg name="use_gazebo" default="false" />
+ <!-- Import Common poperties-->
+    <xacro:include filename="$(find rhacobot_description)/urdf/common_properties.xacro" />
+  <!-- Import Rhacobot mobile base -->
+  <xacro:include filename="$(find rhacobot_description)/urdf/mobile_base.xacro" />
+  <!-- Import Rhacobot tail -->
+  <xacro:include filename="$(find rhacobot_description)/urdf/tail.xacro" />
+  <xacro:if value="$(arg use_gazebo)">
+    <xacro:include filename="$(find rhacobot_gazebo)/xacro/rhacobot.gazebo.xacro" />
+  </xacro:if>
+  <joint name="base_tail_base_joint" type="fixed">
+    <parent link="body_link" />
+    <child link="tail_base_link" />
+    <origin xyz="-0.185 0 -0.0335" rpy="0 0 0" />
+  </joint>
 </robot>
