Commit message: add gps

File: rhacobot_description/urdf/mobile_base.xacro (robot description, xacro)
@@ -10,5 +10,5 @@
     <xacro:property name="wheel_length" value="0.04" />
     <xacro:property name="wheel_offset_origin_y" value="0.05" />
-    <link name="base_link"/>
+    <link name="base_link" />
     <link name="body_link">
         <visual>
@@ -28,5 +28,6 @@
                 rpy="0 0 0" />
         </collision>
-        <xacro:box_inertia m="5.0" l="${gazebo_drift_factor * base_length}" w="${gazebo_drift_factor * base_width}" h="${gazebo_drift_factor * base_height}"
+        <xacro:box_inertia m="5.0" l="${gazebo_drift_factor * base_length}"
+            w="${gazebo_drift_factor * base_width}" h="${gazebo_drift_factor * base_height}"
             xyz="${base_offset_origin_x - (base_length /2)} ${base_offset_origin_y} ${base_offset_origin_z - (base_height/2)}"
             rpy="0 0 0" />
@@ -39,19 +40,19 @@
     <link name="imu_body_link">
         <visual>
-          <geometry>
-            <box size="0.001 0.001 0.001"/>
-          </geometry>
+            <geometry>
+                <box size="0.001 0.001 0.001" />
+            </geometry>
         </visual>
         <collision>
-          <geometry>
-            <box size="0.001 0.001 0.001"/>
-        </geometry>
-      </collision>
+            <geometry>
+                <box size="0.001 0.001 0.001" />
+            </geometry>
+        </collision>
     </link>
-      <joint name="imu_body_joint" type="fixed">
-        <parent link="body_link"/>
-        <child link="imu_body_link"/>
-        <origin xyz="0 0 0.05"/>
-      </joint>
+    <joint name="imu_body_joint" type="fixed">
+        <parent link="body_link" />
+        <child link="imu_body_link" />
+        <origin xyz="0 0 0.05" />
+    </joint>
     <link name="right_wheel_link">
         <visual>
@@ -69,5 +70,6 @@
             <origin xyz="0 -${wheel_offset_origin_y}  0" rpy="${pi / 2.0} 0 0" />
         </collision>
-        <xacro:cylinder_inertia m="1.0" r="${gazebo_drift_factor * wheel_radius}" h="${gazebo_drift_factor * wheel_length}"
+        <xacro:cylinder_inertia m="1.0" r="${gazebo_drift_factor * wheel_radius}"
+            h="${gazebo_drift_factor * wheel_length}"
             xyz="0 -${wheel_offset_origin_y}  0" rpy="${pi / 2.0} 0 0" />
     </link>
@@ -79,21 +81,22 @@
     </joint>
     <link name="left_wheel_link">
-            <visual>
-                <geometry>
-                    <mesh filename="file://$(find rhacobot_description)/meshes/wheel.stl"
-                        scale="0.001 0.001 0.001" />
-                </geometry>
-                <origin xyz="0 0 0" rpy="0 0 0" />
-                <material name="grey" />
-            </visual>
-            <collision>
-                <geometry>
-                    <cylinder radius="${wheel_radius}" length="${wheel_length}" />
-                </geometry>
-                <origin xyz="0 ${wheel_offset_origin_y}  0" rpy="${pi / 2.0} 0 0" />
-            </collision>
-            <xacro:cylinder_inertia m="1.0" r="${gazebo_drift_factor * wheel_radius}" h="${gazebo_drift_factor * wheel_length}"
-                xyz="0 ${wheel_offset_origin_y}  0" rpy="${pi / 2.0} 0 0" />
-        </link>
+        <visual>
+            <geometry>
+                <mesh filename="file://$(find rhacobot_description)/meshes/wheel.stl"
+                    scale="0.001 0.001 0.001" />
+            </geometry>
+            <origin xyz="0 0 0" rpy="0 0 0" />
+            <material name="grey" />
+        </visual>
+        <collision>
+            <geometry>
+                <cylinder radius="${wheel_radius}" length="${wheel_length}" />
+            </geometry>
+            <origin xyz="0 ${wheel_offset_origin_y}  0" rpy="${pi / 2.0} 0 0" />
+        </collision>
+        <xacro:cylinder_inertia m="1.0" r="${gazebo_drift_factor * wheel_radius}"
+            h="${gazebo_drift_factor * wheel_length}"
+            xyz="0 ${wheel_offset_origin_y}  0" rpy="${pi / 2.0} 0 0" />
+    </link>
     <joint name="base_left_wheel_joint" type="continuous">
         <parent link="body_link" />

File: rhacobot_simulation/macros/imu.xacro (robot description, xacro)
@@ -5,5 +5,5 @@
             <sensor name="SimIMU" type="imu">
                 <always_on>1</always_on>
-                <update_rate>25.0</update_rate>
+                <update_rate>${hz}</update_rate>
                 <visualize>true</visualize>
                 <topic>${topic}</topic>

File: rhacobot_simulation/xacro/rhacobot.gazebo.xacro (robot description, xacro)
@@ -3,8 +3,14 @@
     <xacro:arg name="controllers" default="true" />
     <xacro:arg name="imu" default="true" />
+    <xacro:arg name="gps" default="true" />
     <!-- IMU   -->
     <xacro:if value="$(arg imu)">
         <xacro:include filename="$(find rhacobot_simulation)/macros/imu.xacro" />
         <xacro:imu link="imu_body_link" hz="50" topic="imu" />
+    </xacro:if>
+    <!-- GPS   -->
+    <xacro:if value="$(arg gps)">
+        <xacro:include filename="$(find rhacobot_simulation)/macros/gps.xacro" />
+        <xacro:gps link="imu_body_link" hz="50" topic="gps" />
     </xacro:if>
     <!-- Import Rhacobot mobile base -->

Commit message: real case

File: rhacobot_description/urdf/mobile_base.xacro (robot description, xacro)
@@ -85,5 +85,5 @@
         <parent link="base_link" />
         <child link="left_wheel_link" />
-        <origin xyz="0 ${base_width  / 2.0} 0" rpy="0 0 0" />
+        <origin xyz="0 ${base_width  / 2.0} 0" rpy="0 0 ${pi}" />
         <axis xyz="0 1 0" />
     </joint>

File: rhacobot_description/urdf/sensors.xacro (robot description, xacro)
@@ -33,5 +33,5 @@
         <parent link="tail_arm_link" />
         <child link="wt901_link" />
-        <origin xyz="0.17 0.04 -0.008" />
+        <origin xyz="0.17 0.04 -0.008" rpy="0 0 0"  />
     </joint>
     <link name="wt31n_link">
@@ -50,5 +50,5 @@
         <parent link="tail_forearm_link" />
         <child link="wt31n_link" />
-        <origin xyz="0.17 0 0.045" />
+        <origin xyz="0.17 0 0.045" rpy="0 0 0" />
     </joint>
 </robot>

File: rhacobot_description/urdf/tail.xacro (robot description, xacro)
@@ -50,5 +50,5 @@
         <parent link="tail_base_link" />
         <child link="tail_shoulder_link" />
-        <origin xyz="0 0 0" rpy="0 0 ${pi}" />
+        <origin xyz="0 0 0" rpy="0 0 0" />
         <limit effort="100" velocity="100" lower="-${pi/4}" upper="${pi/4}" />
         <axis xyz="0 0 1" />
@@ -76,6 +76,6 @@
         <parent link="tail_shoulder_link" />
         <child link="tail_arm_link" />
-        <origin xyz="0 0 0.079" rpy="0 0 0" />
-        <limit effort="100" velocity="100" lower="-${pi/2}" upper="${pi/6}" />
+        <origin xyz="0 0 0.079" rpy="0 ${pi} 0" />
+        <limit effort="100" velocity="100" lower="${-pi/2 + pi}" upper="${pi/6 + pi}" />
         <axis xyz="0 1 0" />
     </joint>

Commit message: fix tf

File: rhacobot_description/urdf/mobile_base.xacro (robot description, xacro)
@@ -69,5 +69,5 @@
                     scale="0.001 0.001 0.001" />
             </geometry>
-            <origin xyz="0 0 0" rpy="0 0 0" />
+            <origin xyz="0 0 0" rpy="0 0 ${pi}" />
             <material name="grey" />
         </visual>

File: rhacobot_description/urdf/tail.xacro (robot description, xacro)
@@ -50,5 +50,5 @@
         <parent link="tail_base_link" />
         <child link="tail_shoulder_link" />
-        <origin xyz="0 0 0" rpy="0 0 0" />
+        <origin xyz="0 0 0" rpy="0 0 ${pi}" />
         <limit effort="100" velocity="100" lower="-${pi/4}" upper="${pi/4}" />
         <axis xyz="0 0 1" />

Commit message: fix tf  wheel

File: rhacobot_description/urdf/mobile_base.xacro (robot description, xacro)
@@ -69,5 +69,5 @@
                     scale="0.001 0.001 0.001" />
             </geometry>
-            <origin xyz="0 0 0" rpy="0 0 ${pi}" />
+            <origin xyz="0 0 0" rpy="${pi} 0 0" />
             <material name="grey" />
         </visual>
@@ -76,14 +76,14 @@
                 <cylinder radius="${wheel_radius}" length="${wheel_length}" />
             </geometry>
-            <origin xyz="0 ${wheel_offset_origin_y}  0" rpy="${pi / 2.0} 0 0" />
+            <origin xyz="0 -${wheel_offset_origin_y}  0" rpy="${pi / 2.0} 0 0" />
         </collision>
         <xacro:cylinder_inertia m="1.0" r="${gazebo_drift_factor * wheel_radius}"
             h="${gazebo_drift_factor * wheel_length}"
-            xyz="0 ${wheel_offset_origin_y}  0" rpy="${pi / 2.0} 0 0" />
+            xyz="0 -${wheel_offset_origin_y}  0" rpy="${pi / 2.0} 0 0" />
     </link>
     <joint name="base_left_wheel_joint" type="continuous">
         <parent link="base_link" />
         <child link="left_wheel_link" />
-        <origin xyz="0 ${base_width  / 2.0} 0" rpy="0 0 ${pi}" />
+        <origin xyz="0 ${base_width  / 2.0} 0" rpy="${pi} 0 0" />
         <axis xyz="0 1 0" />
     </joint>
