Commit message: fix tail

File: rhacobot_description/urdf/sensors.xacro (robot description, xacro)
@@ -33,5 +33,5 @@
         <parent link="tail_arm_link" />
         <child link="wt901_link" />
-        <origin xyz="0.17 0.04 -0.008" rpy="0 0 0"  />
+        <origin xyz="0.17 -0.04 0.008" rpy="0 0 0"  />
     </joint>
     <link name="wt31n_link">
@@ -50,5 +50,5 @@
         <parent link="tail_forearm_link" />
         <child link="wt31n_link" />
-        <origin xyz="0.17 0 0.045" rpy="0 0 0" />
+        <origin xyz="0.17 0 -0.045" rpy="0 0 0" />
     </joint>
 </robot>

File: rhacobot_description/urdf/tail.xacro (robot description, xacro)
@@ -27,5 +27,5 @@
         <parent link="body_link" />
         <child link="tail_base_link" />
-        <origin xyz="-0.185 0 -0.0335" rpy="0 0 0" />
+        <origin xyz="-0.185 0 -0.0335" rpy="0 0 ${pi}" />
     </joint>
     <link name="tail_shoulder_link">
@@ -50,5 +50,5 @@
         <parent link="tail_base_link" />
         <child link="tail_shoulder_link" />
-        <origin xyz="0 0 0" rpy="0 0 ${pi}" />
+        <origin xyz="0 0 0" rpy="0 0 0" />
         <limit effort="100" velocity="100" lower="-${pi/4}" upper="${pi/4}" />
         <axis xyz="0 0 1" />
@@ -56,5 +56,5 @@
     <link name="tail_arm_link">
         <visual>
-            <origin xyz="0 0 0" rpy="0 0 0" />
+            <origin xyz="0 0 0" rpy="${pi} 0 0" />
             <geometry>
                 <mesh filename="file://$(find rhacobot_description)/meshes/tail_joint_b.stl"
@@ -64,5 +64,5 @@
         </visual>
         <collision>    <!-- tail_joint_c macro -->
-            <origin xyz="0 0 0" rpy="0 0 0" />
+            <origin xyz="0 0 0" rpy="${pi} 0 0" />
             <geometry>
                 <mesh filename="file://$(find rhacobot_description)/meshes/tail_joint_b.stl"
@@ -71,16 +71,16 @@
         </collision>
         <xacro:cylinder_inertia m="1.0" r="${gazebo_drift_factor * arm_radius}" h="${gazebo_drift_factor * arm_length}"
-            xyz="0 0 0" rpy="0 ${pi / 2.0} 0" />
+            xyz="0 0 0" rpy="${pi} ${pi / 2.0} 0" />
     </link>
     <joint name="shoulder_arm_joint" type="revolute">
         <parent link="tail_shoulder_link" />
         <child link="tail_arm_link" />
-        <origin xyz="0 0 0.079" rpy="0 ${pi} ${pi}" />
-        <limit effort="100" velocity="100" lower="${-pi/2 + pi}" upper="${pi/6 + pi}" />
+        <origin xyz="0 0 0.079" rpy="${pi} 0 0" />
+        <limit effort="100" velocity="100" lower="${-pi/6}" upper="${pi/2}" />
         <axis xyz="0 1 0" />
     </joint>
     <link name="tail_forearm_link">
         <visual>
-            <origin xyz="0 0 0" rpy="0 0 0" />
+            <origin xyz="0 0 0" rpy="${pi} 0 0" />
             <geometry>
                 <mesh filename="file://$(find rhacobot_description)/meshes/tail_joint_c.stl"
@@ -90,5 +90,5 @@
         </visual>
         <collision>
-            <origin xyz="0 0 0" rpy="0 0 0" />
+            <origin xyz="0 0 0" rpy="${pi} 0 0" />
             <geometry>
                 <mesh filename="file://$(find rhacobot_description)/meshes/tail_joint_c.stl"
@@ -97,5 +97,5 @@
         </collision>
         <xacro:cylinder_inertia m="1.0" r="${gazebo_drift_factor * arm_radius}" h="${gazebo_drift_factor * arm_length}"
-            xyz="0 0 0" rpy="0 ${pi / 2.0} 0" />
+            xyz="0 0 0" rpy="${pi} ${pi / 2.0} 0" />
     </link>
     <joint name="arm_forearm_joint" type="revolute">
@@ -103,5 +103,5 @@
         <child link="tail_forearm_link" />
         <origin xyz="0.25 0 0" rpy="0 0 0" />
-        <limit effort="100" velocity="100" lower="-${pi/4}" upper="${pi/1.4}" />
+        <limit effort="100" velocity="100" lower="-${pi/1.4}" upper="${pi/4}" />
         <axis xyz="0 1 0" />
     </joint>
@@ -127,5 +127,5 @@
         <parent link="tail_forearm_link" />
         <child link="tail_wheel_link" />
-        <origin xyz="0.257256 0 0.029611" rpy="0 0 0" />
+        <origin xyz="0.257256 0 -0.029611" rpy="0 0 0" />
     </joint>
 </robot>
