Commit message: add ekf

File: rhacobot_control/xacro/tail.ros2_control.xacro (robot description, xacro)
@@ -39,4 +39,5 @@
                     <param name="kp_position">100</param>
                     <param name="ki_position">0.0</param>
+                    <param name="initial_angle_offset">0.0</param>
                 </xacro:unless>
             </joint>
@@ -66,4 +67,5 @@
                     <param name="kp_position">100</param>
                     <param name="ki_position">0.0</param>
+                    <param name="initial_angle_offset">0.0</param>
                 </xacro:unless>
             </joint>
@@ -93,4 +95,5 @@
                     <param name="kp_position">100</param>
                     <param name="ki_position">0.0</param>
+                    <param name="initial_angle_offset">0.0</param>
                 </xacro:unless>
             </joint>

File: rhacobot_description/urdf/mobile_base.xacro (robot description, xacro)
@@ -10,5 +10,4 @@
     <xacro:property name="wheel_length" value="0.04" />
     <xacro:property name="wheel_offset_origin_y" value="0.05" />
-    <link name="base_link" />
     <link name="body_link">
         <visual>
@@ -33,25 +32,9 @@
             rpy="0 0 0" />
     </link>
-    <joint name="base_joint" type="fixed">
+    <joint name="base_body_joint" type="continuous">
         <parent link="base_link" />
         <child link="body_link" />
-        <origin xyz="0 0 ${wheel_radius}" rpy="0 0 0" />
-    </joint>
-    <link name="imu_body_link">
-        <visual>
-            <geometry>
-                <box size="0.001 0.001 0.001" />
-            </geometry>
-        </visual>
-        <collision>
-            <geometry>
-                <box size="0.001 0.001 0.001" />
-            </geometry>
-        </collision>
-    </link>
-    <joint name="imu_body_joint" type="fixed">
-        <parent link="body_link" />
-        <child link="imu_body_link" />
-        <origin xyz="0 0 0.05" />
+        <origin xyz="0 0 0" rpy="0 0 0" />
+        <axis xyz="0 1 0" />
     </joint>
     <link name="right_wheel_link">
@@ -75,5 +58,5 @@
     </link>
     <joint name="base_right_wheel_joint" type="continuous">
-        <parent link="body_link" />
+        <parent link="base_link" />
         <child link="right_wheel_link" />
         <origin xyz="0 -${base_width / 2.0} 0" rpy="0 0 0" />
@@ -100,5 +83,5 @@
     </link>
     <joint name="base_left_wheel_joint" type="continuous">
-        <parent link="body_link" />
+        <parent link="base_link" />
         <child link="left_wheel_link" />
         <origin xyz="0 ${base_width  / 2.0} 0" rpy="0 0 0" />

File: rhacobot_description/urdf/rhacobot.urdf.xacro (robot description, xacro)
@@ -1,24 +1,36 @@
 <?xml version="1.0" encoding="utf-8"?>
 <robot xmlns:xacro="http://www.ros.org/wiki/xacro" name="rhacobot_urdf">
-    <!-- parameters -->
+  <!-- parameters -->
   <xacro:arg name="use_simulation" default="false" />
   <xacro:arg name="use_controllers" default="true" />
- <!-- Import Common poperties-->
-    <xacro:include filename="$(find rhacobot_description)/urdf/common_properties.xacro" />
+ <!-- Import Common properties-->
+  <xacro:include filename="$(find rhacobot_description)/urdf/common_properties.xacro" />
   <!-- Import Rhacobot mobile base -->
   <xacro:include filename="$(find rhacobot_description)/urdf/mobile_base.xacro" />
   <!-- Import Rhacobot tail -->
   <xacro:include filename="$(find rhacobot_description)/urdf/tail.xacro" />
+  <!-- Import Sensors -->
+  <xacro:include filename="$(find rhacobot_description)/urdf/sensors.xacro" />
+  <!-- Import controller manager and hardware interfaces -->
+  <xacro:if value="$(arg use_controllers)">
+    <xacro:include filename="$(find rhacobot_control)/xacro/rhacobot.ros2_control.xacro" />
+  </xacro:if>
+  <!-- Import if use simulation -->
   <xacro:if value="$(arg use_simulation)">
     <xacro:include filename="$(find rhacobot_simulation)/xacro/rhacobot.gazebo.xacro" />
   </xacro:if>
-  <!-- controller manager and hardware interfaces -->
-  <xacro:if value="$(arg use_controllers)">
-    <xacro:include filename="$(find rhacobot_control)/xacro/rhacobot.ros2_control.xacro" />
-  </xacro:if>
-  <joint name="base_tail_base_joint" type="fixed">
-    <parent link="body_link" />
-    <child link="tail_base_link" />
-    <origin xyz="-0.185 0 -0.0335" rpy="0 0 0" />
-  </joint>
+  <link name="base_link">
+    <visual>
+      <geometry>
+          <box size="0.001 0.001 0.001" />
+      </geometry>
+    </visual>
+    <collision>
+        <geometry>
+            <box size="0.001 0.001 0.001" />
+        </geometry>
+    </collision>
+    <xacro:sphere_inertia m="0.0001" r="0.001"
+    xyz="0 0 0" rpy="0 0 0" />
+  </link>
 </robot>

File: rhacobot_description/urdf/tail.xacro (robot description, xacro)
@@ -24,4 +24,9 @@
             xyz="0 0 0" rpy="0 0 0" />
     </link>
+    <joint name="body_tail_base_joint" type="fixed">
+        <parent link="body_link" />
+        <child link="tail_base_link" />
+        <origin xyz="-0.185 0 -0.0335" rpy="0 0 0" />
+    </joint>
     <link name="tail_shoulder_link">
         <visual>

File: rhacobot_simulation/macros/imu.xacro (robot description, xacro)
@@ -1,13 +1,13 @@
 <?xml version="1.0"?>
 <robot xmlns:xacro="http://www.ros.org/wiki/xacro" name="IMU" description="IMU sensor">
-    <xacro:macro name="imu" params="link hz topic">
-        <gazebo reference="${link}">
-            <sensor name="SimIMU" type="imu">
+    <xacro:macro name="imu" params="name hz topic">
+        <gazebo reference="${name}_link">
+            <sensor name="${name}_imu" type="imu">
                 <always_on>1</always_on>
                 <update_rate>${hz}</update_rate>
                 <visualize>true</visualize>
                 <topic>${topic}</topic>
-                <frame_id>${link}</frame_id>
-                <ignition_frame_id>${link}</ignition_frame_id>
+                <frame_id>${name}_link</frame_id>
+                <ignition_frame_id>${name}_link</ignition_frame_id>
                 <imu>
                     <orientation_reference_frame>

File: rhacobot_simulation/xacro/rhacobot.gazebo.xacro (robot description, xacro)
@@ -1,18 +1,40 @@
 <?xml version="1.0" encoding="utf-8"?>
 <robot xmlns:xacro="http://www.ros.org/wiki/xacro">
-    <xacro:arg name="imu" default="true" />
-    <xacro:arg name="gps" default="false" />
+    <xacro:arg name="use_imu" default="true" />
+    <xacro:arg name="use_mag" default="true" />
+    <xacro:arg name="use_gps" default="true" />
     <!-- IMU   -->
-    <xacro:if value="$(arg imu)">
+    <xacro:if value="$(arg use_imu)">
+        <gazebo>
+            <plugin filename="libignition-gazebo-imu-system.so"
+                    name="ignition::gazebo::systems::Imu">
+            </plugin>
+        </gazebo>
         <xacro:include filename="$(find rhacobot_simulation)/macros/imu.xacro" />
-        <xacro:imu link="imu_body_link" hz="50" topic="imu" />
+        <xacro:imu name="wtgahrs1" hz="50" topic="imu/wtgahrs1" />
+        <xacro:imu name="wt901" hz="50" topic="imu/wt901" />
+        <xacro:imu name="wt31n" hz="50" topic="imu/wt31n" />
     </xacro:if>
-    <!-- GPS   -->
-    <xacro:if value="$(arg gps)">
+    <!-- MAG   -->
+    <xacro:if value="$(arg use_mag)">
+        <gazebo>
+            <plugin filename="ignition-gazebo-magnetometer-system"
+                name="gz::sim::systems::Magnetometer">
+            </plugin>
+        </gazebo>
+        <xacro:include filename="$(find rhacobot_simulation)/macros/mag.xacro" />
+        <xacro:mag name="wtgahrs1" hz="50" topic="mag/wtgahrs1" />
+        <xacro:mag name="wt901" hz="50" topic="mag/wt901" />
+    </xacro:if>
+     <!-- GPS   -->
+    <xacro:if value="$(arg use_gps)">
+        <gazebo>
+            <plugin filename="ignition-gazebo-navsat-system"
+                    name="ignition::gazebo::systems::NavSat">
+            </plugin>
+        </gazebo>
         <xacro:include filename="$(find rhacobot_simulation)/macros/gps.xacro" />
-        <xacro:gps link="imu_body_link" hz="50" topic="gps/fix" />
+        <xacro:gps name="wtgahrs1" hz="50" topic="gps/wtgahrs1/fix" />
     </xacro:if>
-    <!-- Import Rhacobot mobile base -->
-    <xacro:include filename="$(find rhacobot_simulation)/xacro/mobile_base.gazebo.xacro" />
     <!-- Import Rhacobot tail -->
     <xacro:include filename="$(find rhacobot_simulation)/xacro/tail.gazebo.xacro" />
