Commit message: upgrade gazebo_classic -> gazebo_fortress

File: rhacobot_control/xacro/mobile_base.ros2_control.xacro (robot description, xacro)
@@ -1,11 +1,11 @@
 <?xml version="1.0" ?>
 <robot xmlns:xacro="http://www.ros.org/wiki/xacro" >
-    <xacro:macro name="mobile_base_ros2_control" params="ifname use_gazebo:=^|false">
+    <xacro:macro name="mobile_base_ros2_control" params="ifname use_simulation:=^|false">
         <ros2_control name="mobile_base_ros2_control" type="system">
             <hardware>
-                <xacro:if value="${use_gazebo}">
-                    <plugin>gazebo_ros2_control/GazeboSystem</plugin>
+                <xacro:if value="${use_simulation}">
+                    <plugin>ign_ros2_control/IgnitionSystem</plugin>
                 </xacro:if>
-                <xacro:unless value="${use_gazebo}">
+                <xacro:unless value="${use_simulation}">
                     <plugin>myactuator_hardware_interface/MyActuatorHardwareInterface</plugin>
                     <param name="ifname">${ifname}</param>
@@ -15,10 +15,10 @@
             </hardware>
             <joint name="base_left_wheel_joint">
-                <xacro:if value="${use_gazebo}">
+                <xacro:if value="${use_simulation}">
                     <command_interface name="velocity"/>
                     <state_interface name="position"/>
                     <state_interface name="velocity"/>
                 </xacro:if>
-                <xacro:unless value="${use_gazebo}">
+                <xacro:unless value="${use_simulation}">
                     <param name="can_id">1</param>
                     <param name="reducer_ratio">6.2</param>
@@ -39,10 +39,10 @@
             </joint>
             <joint name="base_right_wheel_joint">
-                <xacro:if value="${use_gazebo}">
+                <xacro:if value="${use_simulation}">
                     <command_interface name="velocity"/>
                     <state_interface name="position"/>
                     <state_interface name="velocity"/>
                 </xacro:if>
-                <xacro:unless value="${use_gazebo}">
+                <xacro:unless value="${use_simulation}">
                     <param name="can_id">2</param>
                     <param name="reducer_ratio">6.2</param>

File: rhacobot_control/xacro/rhacobot.ros2_control.xacro (robot description, xacro)
@@ -5,5 +5,5 @@
   <xacro:include filename="$(find rhacobot_control)/xacro/mobile_base.ros2_control.xacro" />
   <xacro:include filename="$(find rhacobot_control)/xacro/tail.ros2_control.xacro" />
-  <xacro:mobile_base_ros2_control ifname="$(arg ifname)" use_gazebo="$(arg use_gazebo)"/>
-  <xacro:tail_ros2_control ifname="$(arg ifname)" use_gazebo="$(arg use_gazebo)"/>
+  <xacro:mobile_base_ros2_control ifname="$(arg ifname)" use_simulation="$(arg use_simulation)"/>
+  <xacro:tail_ros2_control ifname="$(arg ifname)" use_simulation="$(arg use_simulation)"/>
 </robot>

File: rhacobot_control/xacro/tail.ros2_control.xacro (robot description, xacro)
@@ -1,11 +1,11 @@
 <?xml version="1.0"?>
 <robot xmlns:xacro="http://www.ros.org/wiki/xacro">
-    <xacro:macro name="tail_ros2_control" params="ifname use_gazebo:=^|false">
+    <xacro:macro name="tail_ros2_control" params="ifname use_simulation:=^|false">
         <ros2_control name="tail_ros2_control" type="system">
             <hardware>
-                <xacro:if value="${use_gazebo}">
-                    <plugin>gazebo_ros2_control/GazeboSystem</plugin>
+                <xacro:if value="${use_simulation}">
+                    <plugin>ign_ros2_control/IgnitionSystem</plugin>
                 </xacro:if>
-                <xacro:unless value="${use_gazebo}">
+                <xacro:unless value="${use_simulation}">
                     <plugin>myactuator_hardware_interface/MyActuatorHardwareInterface</plugin>
                     <param name="ifname">${ifname}</param>
@@ -15,5 +15,5 @@
             </hardware>
             <joint name="tail_base_shoulder_joint">
-                <xacro:if value="${use_gazebo}">
+                <xacro:if value="${use_simulation}">
                     <command_interface name="position">
                         <param name="min">-1</param>
@@ -23,5 +23,5 @@
                     <state_interface name="velocity" />
                 </xacro:if>
-                <xacro:unless value="${use_gazebo}">
+                <xacro:unless value="${use_simulation}">
                     <param name="can_id">3</param>
                     <param name="reducer_ratio">6.2</param>
@@ -42,5 +42,5 @@
             </joint>
             <joint name="shoulder_arm_joint">
-                <xacro:if value="${use_gazebo}">
+                <xacro:if value="${use_simulation}">
                     <command_interface name="position">
                         <param name="min">-1</param>
@@ -50,5 +50,5 @@
                     <state_interface name="velocity" />
                 </xacro:if>
-                <xacro:unless value="${use_gazebo}">
+                <xacro:unless value="${use_simulation}">
                     <param name="can_id">4</param>
                     <param name="reducer_ratio">6.2</param>
@@ -69,5 +69,5 @@
             </joint>
             <joint name="arm_forearm_joint">
-                <xacro:if value="${use_gazebo}">
+                <xacro:if value="${use_simulation}">
                     <command_interface name="position">
                         <param name="min">-1</param>
@@ -77,5 +77,5 @@
                     <state_interface name="velocity" />
                 </xacro:if>
-                <xacro:unless value="${use_gazebo}">
+                <xacro:unless value="${use_simulation}">
                     <param name="can_id">5</param>
                     <param name="reducer_ratio">6.2</param>

File: rhacobot_description/urdf/common_properties.xacro (robot description, xacro)
@@ -1,5 +1,5 @@
 <?xml version="1.0"?>
 <robot xmlns:xacro="http://www.ros.org/wiki/xacro">
-    <xacro:property name="gazebo_drift_factor" value="6" />
+    <xacro:property name="gazebo_drift_factor" value="1" />
     <material name="silver">
         <color rgba="0.700 0.700 0.700 1.000" />

File: rhacobot_description/urdf/rhacobot.urdf.xacro (robot description, xacro)
@@ -2,5 +2,5 @@
 <robot xmlns:xacro="http://www.ros.org/wiki/xacro" name="rhacobot_urdf">
     <!-- parameters -->
-  <xacro:arg name="use_gazebo" default="false" />
+  <xacro:arg name="use_simulation" default="false" />
  <!-- Import Common poperties-->
     <xacro:include filename="$(find rhacobot_description)/urdf/common_properties.xacro" />
@@ -9,6 +9,6 @@
   <!-- Import Rhacobot tail -->
   <xacro:include filename="$(find rhacobot_description)/urdf/tail.xacro" />
-  <xacro:if value="$(arg use_gazebo)">
-    <xacro:include filename="$(find rhacobot_gazebo)/xacro/rhacobot.gazebo.xacro" />
+  <xacro:if value="$(arg use_simulation)">
+    <xacro:include filename="$(find rhacobot_simulation)/xacro/rhacobot.gazebo.xacro" />
   </xacro:if>
   <joint name="base_tail_base_joint" type="fixed">

File: rhacobot_simulation/xacro/rhacobot.gazebo.xacro (robot description, xacro)
@@ -5,15 +5,15 @@
     <!-- IMU   -->
     <xacro:if value="$(arg imu)">
-        <xacro:include filename="$(find rhacobot_gazebo)/macros/imu.xacro" />
+        <xacro:include filename="$(find rhacobot_simulation)/macros/imu.xacro" />
         <xacro:imu link="imu_body_link" hz="50" topic="IMU" />
     </xacro:if>
     <!-- Import Rhacobot mobile base -->
-    <xacro:include filename="$(find rhacobot_gazebo)/xacro/mobile_base.gazebo.xacro" />
+    <xacro:include filename="$(find rhacobot_simulation)/xacro/mobile_base.gazebo.xacro" />
     <!-- Import Rhacobot tail -->
-    <xacro:include filename="$(find rhacobot_gazebo)/xacro/tail.gazebo.xacro" />
+    <xacro:include filename="$(find rhacobot_simulation)/xacro/tail.gazebo.xacro" />
     <!-- controller manager and hardware interfaces -->
     <xacro:if value="$(arg controllers)">
         <gazebo>
-            <plugin filename="libgazebo_ros2_control.so" name="gazebo_ros2_control">
+            <plugin filename="ign_ros2_control-system" name="ign_ros2_control::IgnitionROS2ControlPlugin">
                 <parameters>$(find rhacobot_control)/config/controllers.yaml</parameters>
             </plugin>

Commit message: test1

File: rhacobot_control/xacro/mobile_base.ros2_control.xacro (robot description, xacro)
@@ -36,4 +36,5 @@
                     <param name="kp_position">100</param>
                     <param name="ki_position">0</param>
+                    <param name="initial_angle_offset">0.0</param>
                 </xacro:unless>
             </joint>
@@ -60,4 +61,5 @@
                     <param name="kp_position">100</param>
                     <param name="ki_position">0.0</param>
+                    <param name="initial_angle_offset">0.0</param>
                 </xacro:unless>
             </joint>

File: rhacobot_control/xacro/tail.ros2_control.xacro (robot description, xacro)
@@ -39,4 +39,5 @@
                     <param name="kp_position">100</param>
                     <param name="ki_position">0.0</param>
+                    <param name="initial_angle_offset">0.0</param>
                 </xacro:unless>
             </joint>
@@ -47,5 +48,7 @@
                         <param name="max">1</param>
                     </command_interface>
-                    <state_interface name="position" />
+                    <state_interface name="position">
+                        <param name="initial_value">0.0</param>
+                    </state_interface>
                     <state_interface name="velocity" />
                 </xacro:if>
@@ -66,4 +69,5 @@
                     <param name="kp_position">100</param>
                     <param name="ki_position">0.0</param>
+                    <param name="initial_angle_offset">0.0</param>
                 </xacro:unless>
             </joint>
@@ -93,4 +97,5 @@
                     <param name="kp_position">100</param>
                     <param name="ki_position">0.0</param>
+                    <param name="initial_angle_offset">0.0</param>
                 </xacro:unless>
             </joint>

File: rhacobot_description/urdf/mobile_base.xacro (robot description, xacro)
@@ -10,5 +10,4 @@
     <xacro:property name="wheel_length" value="0.04" />
     <xacro:property name="wheel_offset_origin_y" value="0.05" />
-    <link name="base_link" />
     <link name="body_link">
         <visual>
@@ -33,25 +32,8 @@
             rpy="0 0 0" />
     </link>
-    <joint name="base_joint" type="fixed">
+    <joint name="base_body_joint" type="fixed">
         <parent link="base_link" />
         <child link="body_link" />
-        <origin xyz="0 0 ${wheel_radius}" rpy="0 0 0" />
-    </joint>
-    <link name="imu_body_link">
-        <visual>
-            <geometry>
-                <box size="0.001 0.001 0.001" />
-            </geometry>
-        </visual>
-        <collision>
-            <geometry>
-                <box size="0.001 0.001 0.001" />
-            </geometry>
-        </collision>
-    </link>
-    <joint name="imu_body_joint" type="fixed">
-        <parent link="body_link" />
-        <child link="imu_body_link" />
-        <origin xyz="0 0 0.05" />
+        <origin xyz="0 0 0" rpy="0 0 0" />
     </joint>
     <link name="right_wheel_link">
@@ -75,5 +57,5 @@
     </link>
     <joint name="base_right_wheel_joint" type="continuous">
-        <parent link="body_link" />
+        <parent link="base_link" />
         <child link="right_wheel_link" />
         <origin xyz="0 -${base_width / 2.0} 0" rpy="0 0 0" />
@@ -100,5 +82,5 @@
     </link>
     <joint name="base_left_wheel_joint" type="continuous">
-        <parent link="body_link" />
+        <parent link="base_link" />
         <child link="left_wheel_link" />
         <origin xyz="0 ${base_width  / 2.0} 0" rpy="0 0 0" />

File: rhacobot_description/urdf/rhacobot.urdf.xacro (robot description, xacro)
@@ -1,5 +1,6 @@
 <?xml version="1.0" encoding="utf-8"?>
 <robot xmlns:xacro="http://www.ros.org/wiki/xacro" name="rhacobot_urdf">
-    <!-- parameters -->
+  <!-- parameters -->
+  <xacro:arg name="use_sensors" default="true" />
   <xacro:arg name="use_simulation" default="false" />
   <xacro:arg name="use_controllers" default="true" />
@@ -10,4 +11,7 @@
   <!-- Import Rhacobot tail -->
   <xacro:include filename="$(find rhacobot_description)/urdf/tail.xacro" />
+  <xacro:if value="$(arg use_sensors)">
+    <xacro:include filename="$(find rhacobot_description)/urdf/sensors.xacro" />
+  </xacro:if>
   <xacro:if value="$(arg use_simulation)">
     <xacro:include filename="$(find rhacobot_simulation)/xacro/rhacobot.gazebo.xacro" />
@@ -17,8 +21,4 @@
     <xacro:include filename="$(find rhacobot_control)/xacro/rhacobot.ros2_control.xacro" />
   </xacro:if>
-  <joint name="base_tail_base_joint" type="fixed">
-    <parent link="body_link" />
-    <child link="tail_base_link" />
-    <origin xyz="-0.185 0 -0.0335" rpy="0 0 0" />
-  </joint>
+  <link name="base_link" />
 </robot>

File: rhacobot_description/urdf/tail.xacro (robot description, xacro)
@@ -24,4 +24,9 @@
             xyz="0 0 0" rpy="0 0 0" />
     </link>
+    <joint name="base_tail_base_joint" type="fixed">
+        <parent link="base_link" />
+        <child link="tail_base_link" />
+        <origin xyz="-0.185 0 -0.0335" rpy="0 0 0" />
+    </joint>
     <link name="tail_shoulder_link">
         <visual>

File: rhacobot_simulation/macros/gps.xacro (robot description, xacro)
@@ -1,12 +1,12 @@
 <?xml version="1.0"?>
 <robot xmlns:xacro="http://www.ros.org/wiki/xacro" name="GPS" description="GPS sensor">
-    <xacro:macro name="gps" params="link hz topic">
-        <gazebo reference="${link}">
-            <sensor name="GazeboNavSat" type="navsat">
+    <xacro:macro name="gps" params="name hz topic">
+        <gazebo reference="${name}_link">
+            <sensor name="${name}_gps" type="navsat">
                 <always_on>1</always_on>
                 <update_rate>${hz}</update_rate>
                 <visualize>true</visualize>
                 <topic>${topic}</topic>
-                <ignition_frame_id>${link}</ignition_frame_id>
+                <ignition_frame_id>${name}_link</ignition_frame_id>
             </sensor>
         </gazebo>

File: rhacobot_simulation/macros/imu.xacro (robot description, xacro)
@@ -1,13 +1,13 @@
 <?xml version="1.0"?>
 <robot xmlns:xacro="http://www.ros.org/wiki/xacro" name="IMU" description="IMU sensor">
-    <xacro:macro name="imu" params="link hz topic">
-        <gazebo reference="${link}">
-            <sensor name="SimIMU" type="imu">
+    <xacro:macro name="imu" params="name hz topic">
+        <gazebo reference="${name}_link">
+            <sensor name="${name}_imu" type="imu">
                 <always_on>1</always_on>
                 <update_rate>${hz}</update_rate>
                 <visualize>true</visualize>
                 <topic>${topic}</topic>
-                <frame_id>${link}</frame_id>
-                <ignition_frame_id>${link}</ignition_frame_id>
+                <frame_id>${name}_link</frame_id>
+                <ignition_frame_id>${name}_link</ignition_frame_id>
                 <imu>
                     <orientation_reference_frame>
@@ -18,3 +18,36 @@
         </gazebo>
     </xacro:macro>
+    <xacro:macro name="mag" params="name hz topic">
+        <gazebo reference="${name}_link">
+            <sensor name="${name}_mag" type="magnetometer">
+                <always_on>1</always_on>
+                <update_rate>${hz}</update_rate>
+                <visualize>true</visualize>
+                <topic>${topic}</topic>
+                <frame_id>${name}_link</frame_id>
+                <ignition_frame_id>${name}_link</ignition_frame_id>
+                <enable_metrics>true</enable_metrics>
+                <magnetometer>
+                  <x>
+                    <noise type="gaussian">
+                      <mean>0.0</mean>
+                      <stddev>0.1</stddev>
+                    </noise>
+                  </x>
+                  <y>
+                    <noise type="gaussian">
+                      <mean>0.0</mean>
+                      <stddev>0.1</stddev>
+                    </noise>
+                  </y>
+                  <z>
+                    <noise type="gaussian">
+                      <mean>0.0</mean>
+                      <stddev>0.1</stddev>
+                    </noise>
+                  </z>
+                </magnetometer>
+              </sensor>
+        </gazebo>
+    </xacro:macro>
 </robot>

File: rhacobot_simulation/xacro/rhacobot.gazebo.xacro (robot description, xacro)
@@ -1,15 +1,41 @@
 <?xml version="1.0" encoding="utf-8"?>
 <robot xmlns:xacro="http://www.ros.org/wiki/xacro">
-    <xacro:arg name="imu" default="true" />
-    <xacro:arg name="gps" default="false" />
-    <!-- IMU   -->
-    <xacro:if value="$(arg imu)">
-        <xacro:include filename="$(find rhacobot_simulation)/macros/imu.xacro" />
-        <xacro:imu link="imu_body_link" hz="50" topic="imu" />
-    </xacro:if>
-    <!-- GPS   -->
-    <xacro:if value="$(arg gps)">
-        <xacro:include filename="$(find rhacobot_simulation)/macros/gps.xacro" />
-        <xacro:gps link="imu_body_link" hz="50" topic="gps/fix" />
+    <xacro:arg name="use_imu" default="true" />
+    <xacro:arg name="use_mag" default="true" />
+    <xacro:arg name="use_gps" default="true" />
+    <xacro:if value="$(arg use_sensors)">
+        <!-- IMU   -->
+        <xacro:if value="$(arg use_imu)">
+            <gazebo>
+                <plugin filename="libignition-gazebo-imu-system.so"
+                        name="ignition::gazebo::systems::Imu">
+                </plugin>
+            </gazebo>
+            <xacro:include filename="$(find rhacobot_simulation)/macros/imu.xacro" />
+            <xacro:imu name="wtgahrs1" hz="50" topic="imu/wtgahrs1" />
+            <xacro:imu name="wt901" hz="50" topic="imu/wt901" />
+            <xacro:imu name="wt31n" hz="50" topic="imu/wt31n" />
+        </xacro:if>
+        <!-- MAG   -->
+        <xacro:if value="$(arg use_mag)">
+            <gazebo>
+                <plugin filename="ignition-gazebo-magnetometer-system"
+                    name="gz::sim::systems::Magnetometer">
+                </plugin>
+            </gazebo>
+            <xacro:include filename="$(find rhacobot_simulation)/macros/imu.xacro" />
+            <xacro:mag name="wtgahrs1" hz="50" topic="mag/wtgahrs1" />
+            <xacro:mag name="wt901" hz="50" topic="mag/wt901" />
+        </xacro:if>
+        <!-- GPS   -->
+        <xacro:if value="$(arg use_gps)">
+            <gazebo>
+                <plugin filename="ignition-gazebo-navsat-system"
+                     name="ignition::gazebo::systems::NavSat">
+                </plugin>
+            </gazebo>
+            <xacro:include filename="$(find rhacobot_simulation)/macros/gps.xacro" />
+            <xacro:gps name="wtgahrs1" hz="50" topic="gps/wtgahrs1/fix" />
+        </xacro:if>
     </xacro:if>
     <!-- Import Rhacobot mobile base -->
