Commit message: use 2bt Hardware interface

File: rhacobot_control/xacro/mobile_base.ros2_control.xacro (robot description, xacro)
@@ -1,68 +1,19 @@
-<?xml version="1.0" ?>
-<robot xmlns:xacro="http://www.ros.org/wiki/xacro" >
-    <xacro:macro name="mobile_base_ros2_control" params="ifname use_simulation:=^|false">
-        <ros2_control name="mobile_base_ros2_control" type="system">
-            <hardware>
-                <xacro:if value="${use_simulation}">
-                    <plugin>ign_ros2_control/IgnitionSystem</plugin>
-                </xacro:if>
-                <xacro:unless value="${use_simulation}">
-                    <plugin>myactuator_hardware_interface/MyActuatorHardwareInterface</plugin>
-                    <param name="ifname">${ifname}</param>
-                    <param name="timeout">1000</param>
-                    <param name="max_speed">5000</param>
-                </xacro:unless>
-            </hardware>
-            <joint name="base_left_wheel_joint">
-                <xacro:if value="${use_simulation}">
-                    <command_interface name="velocity"/>
-                    <state_interface name="position"/>
-                    <state_interface name="velocity"/>
-                </xacro:if>
-                <xacro:unless value="${use_simulation}">
-                    <param name="can_id">1</param>
-                    <param name="reducer_ratio">6.2</param>
-                    <param name="speed_constant">30</param>
-                    <param name="torque_constant">0.29</param>
-                    <param name="rotor_inertia">3400</param>
-                    <param name="position_acceleration">20000</param>
-                    <param name="position_deceleration">20000</param>
-                    <param name="velocity_acceleration">20000</param>
-                    <param name="velocity_deceleration">20000</param>
-                    <param name="kp_current">100</param>
-                    <param name="ki_current">100</param>
-                    <param name="kp_speed">100</param>
-                    <param name="ki_speed">50</param>
-                    <param name="kp_position">100</param>
-                    <param name="ki_position">0</param>
-                    <param name="initial_angle_offset">0.0</param>
-                </xacro:unless>
-            </joint>
-            <joint name="base_right_wheel_joint">
-                <xacro:if value="${use_simulation}">
-                    <command_interface name="velocity"/>
-                    <state_interface name="position"/>
-                    <state_interface name="velocity"/>
-                </xacro:if>
-                <xacro:unless value="${use_simulation}">
-                    <param name="can_id">2</param>
-                    <param name="reducer_ratio">6.2</param>
-                    <param name="speed_constant">30</param>
-                    <param name="torque_constant">0.29</param>
-                    <param name="rotor_inertia">3400</param>
-                    <param name="position_acceleration">20000</param>
-                    <param name="position_deceleration">20000</param>
-                    <param name="velocity_acceleration">20000</param>
-                    <param name="velocity_deceleration">20000</param>
-                    <param name="kp_current">100</param>
-                    <param name="ki_current">100</param>
-                    <param name="kp_speed">100</param>
-                    <param name="ki_speed">50</param>
-                    <param name="kp_position">100</param>
-                    <param name="ki_position">0.0</param>
-                    <param name="initial_angle_offset">0.0</param>
-                </xacro:unless>
-            </joint>
-        </ros2_control>
+<?xml version="1.0"?>
+<robot xmlns:xacro="http://www.ros.org/wiki/xacro">
+    <xacro:arg name="velocity_alpha" default="0.4" />
+    <xacro:arg name="effort_alpha" default="0.4" />
+    <xacro:arg name="torque_constant" default="2.6" />
+    <!-- Import ros2_control -->
+    <xacro:include filename="$(find myactuator_rmd_description)/urdf/myactuator_rmd.ros2_control.xacro" />
+    <xacro:macro name="mobile_base_ros2_control" params="prefix ifname use_simulation:=^|false">
+    <!-- ros2_control configuration -->
+    <xacro:myactuator_rmd_ros2_control name="${prefix}base_left_wheel_ros2_control" joint_name="${prefix}base_left_wheel_joint" simulation="${use_simulation}"
+                                       ifname="${ifname}" actuator_id="3"
+                                       velocity_alpha="$(arg velocity_alpha)" effort_alpha="$(arg effort_alpha)"
+                                       torque_constant="$(arg torque_constant)"/>
+    <xacro:myactuator_rmd_ros2_control name="${prefix}base_right_wheel_ros2_control" joint_name="${prefix}base_right_wheel_joint" simulation="${use_simulation}"
+                                       ifname="${ifname}" actuator_id="4"
+                                       velocity_alpha="$(arg velocity_alpha)" effort_alpha="$(arg effort_alpha)"
+                                       torque_constant="$(arg torque_constant)"/>
     </xacro:macro>
 </robot>

File: rhacobot_control/xacro/rhacobot.ros2_control.xacro (robot description, xacro)
@@ -5,5 +5,5 @@
   <xacro:include filename="$(find rhacobot_control)/xacro/mobile_base.ros2_control.xacro" />
   <xacro:include filename="$(find rhacobot_control)/xacro/tail.ros2_control.xacro" />
-  <xacro:mobile_base_ros2_control ifname="$(arg ifname)" use_simulation="$(arg use_simulation)"/>
-  <xacro:tail_ros2_control ifname="$(arg ifname)" use_simulation="$(arg use_simulation)"/>
+  <xacro:mobile_base_ros2_control prefix="" ifname="$(arg ifname)" use_simulation="$(arg use_simulation)"/>
+  <xacro:tail_ros2_control prefix="" ifname="$(arg ifname)" use_simulation="$(arg use_simulation)"/>
 </robot>

File: rhacobot_control/xacro/tail.ros2_control.xacro (robot description, xacro)
@@ -1,102 +1,23 @@
 <?xml version="1.0"?>
 <robot xmlns:xacro="http://www.ros.org/wiki/xacro">
-    <xacro:macro name="tail_ros2_control" params="ifname use_simulation:=^|false">
-        <ros2_control name="tail_ros2_control" type="system">
-            <hardware>
-                <xacro:if value="${use_simulation}">
-                    <plugin>ign_ros2_control/IgnitionSystem</plugin>
-                </xacro:if>
-                <xacro:unless value="${use_simulation}">
-                    <plugin>myactuator_hardware_interface/MyActuatorHardwareInterface</plugin>
-                    <param name="ifname">${ifname}</param>
-                    <param name="timeout">1000</param>
-                    <param name="max_speed">5000</param>
-                </xacro:unless>
-            </hardware>
-            <joint name="tail_base_shoulder_joint">
-                <xacro:if value="${use_simulation}">
-                    <command_interface name="position">
-                        <param name="min">-1</param>
-                        <param name="max">1</param>
-                    </command_interface>
-                    <state_interface name="position" />
-                    <state_interface name="velocity" />
-                </xacro:if>
-                <xacro:unless value="${use_simulation}">
-                    <param name="can_id">3</param>
-                    <param name="reducer_ratio">6.2</param>
-                    <param name="speed_constant">30</param>
-                    <param name="torque_constant">0.29</param>
-                    <param name="rotor_inertia">3400</param>
-                    <param name="position_acceleration">20000</param>
-                    <param name="position_deceleration">20000</param>
-                    <param name="velocity_acceleration">20000</param>
-                    <param name="velocity_deceleration">20000</param>
-                    <param name="kp_current">100</param>
-                    <param name="ki_current">100</param>
-                    <param name="kp_speed">100</param>
-                    <param name="ki_speed">50</param>
-                    <param name="kp_position">100</param>
-                    <param name="ki_position">0.0</param>
-                    <param name="initial_angle_offset">0.0</param>
-                </xacro:unless>
-            </joint>
-            <joint name="shoulder_arm_joint">
-                <xacro:if value="${use_simulation}">
-                    <command_interface name="position">
-                        <param name="min">-1</param>
-                        <param name="max">1</param>
-                    </command_interface>
-                    <state_interface name="position" />
-                    <state_interface name="velocity" />
-                </xacro:if>
-                <xacro:unless value="${use_simulation}">
-                    <param name="can_id">4</param>
-                    <param name="reducer_ratio">6.2</param>
-                    <param name="speed_constant">30</param>
-                    <param name="torque_constant">0.29</param>
-                    <param name="rotor_inertia">3400</param>
-                    <param name="position_acceleration">20000</param>
-                    <param name="position_deceleration">20000</param>
-                    <param name="velocity_acceleration">20000</param>
-                    <param name="velocity_deceleration">20000</param>
-                    <param name="kp_current">100</param>
-                    <param name="ki_current">100</param>
-                    <param name="kp_speed">100</param>
-                    <param name="ki_speed">50</param>
-                    <param name="kp_position">100</param>
-                    <param name="ki_position">0.0</param>
-                    <param name="initial_angle_offset">0.0</param>
-                </xacro:unless>
-            </joint>
-            <joint name="arm_forearm_joint">
-                <xacro:if value="${use_simulation}">
-                    <command_interface name="position">
-                        <param name="min">-1</param>
-                        <param name="max">1</param>
-                    </command_interface>
-                    <state_interface name="position" />
-                    <state_interface name="velocity" />
-                </xacro:if>
-                <xacro:unless value="${use_simulation}">
-                    <param name="can_id">5</param>
-                    <param name="reducer_ratio">6.2</param>
-                    <param name="speed_constant">30</param>
-                    <param name="torque_constant">0.29</param>
-                    <param name="rotor_inertia">3400</param>
-                    <param name="position_acceleration">20000</param>
-                    <param name="position_deceleration">20000</param>
-                    <param name="velocity_acceleration">20000</param>
-                    <param name="velocity_deceleration">20000</param>
-                    <param name="kp_current">100</param>
-                    <param name="ki_current">100</param>
-                    <param name="kp_speed">100</param>
-                    <param name="ki_speed">50</param>
-                    <param name="kp_position">100</param>
-                    <param name="ki_position">0.0</param>
-                    <param name="initial_angle_offset">0.0</param>
-                </xacro:unless>
-            </joint>
-        </ros2_control>
+    <xacro:arg name="velocity_alpha" default="0.4" />
+    <xacro:arg name="effort_alpha" default="0.4" />
+    <xacro:arg name="torque_constant" default="2.6" />
+    <!-- Import ros2_control -->
+    <xacro:include filename="$(find myactuator_rmd_description)/urdf/myactuator_rmd.ros2_control.xacro" />
+    <xacro:macro name="tail_ros2_control" params="prefix ifname use_simulation:=^|false">
+    <!-- ros2_control configuration -->
+    <xacro:myactuator_rmd_ros2_control name="${prefix}tail_base_shoulder_ros2_control" joint_name="${prefix}tail_base_shoulder_joint" simulation="${use_simulation}"
+                                       ifname="${ifname}" actuator_id="3"
+                                       velocity_alpha="$(arg velocity_alpha)" effort_alpha="$(arg effort_alpha)"
+                                       torque_constant="$(arg torque_constant)"/>
+    <xacro:myactuator_rmd_ros2_control name="${prefix}shoulder_arm_ros2_control" joint_name="${prefix}shoulder_arm_joint" simulation="${use_simulation}"
+                                       ifname="${ifname}" actuator_id="4"
+                                       velocity_alpha="$(arg velocity_alpha)" effort_alpha="$(arg effort_alpha)"
+                                       torque_constant="$(arg torque_constant)"/>
+    <xacro:myactuator_rmd_ros2_control name="${prefix}arm_forearm_ros2_control" joint_name="${prefix}arm_forearm_joint" simulation="${use_simulation}"
+                                       ifname="${ifname}" actuator_id="5"
+                                       velocity_alpha="$(arg velocity_alpha)" effort_alpha="$(arg effort_alpha)"
+                                       torque_constant="$(arg torque_constant)"/>
     </xacro:macro>
 </robot>
